File: kicad/coin_fuyouki.kicad_pcb (KiCad board)
At the start: 2 copper layers, 60 x 70 mm, 58 parts, among them SW1 TACT, U1 PIC16F1503-I/P, U2 AP63205, U3 PC817, U4 PC817, U5-8 TLP291-4

Commit message: Add files via upload
Other:
- board text added: "A4_POLARITY_SILK_v15-42b"
- board text removed: "A4_POLARITY_SILK_v15-42"
Changed lines of the file:
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@@
  (gr_line (start 100 148.5) (end 100 81.5) (stroke (width 0.1) (type default)) (layer "Edge.Cuts"))
  (gr_arc (start 100 81.5) (mid 100.4393 80.4393) (end 101.5 80) (stroke (width 0.1) (type default)) (layer "Edge.Cuts"))
- (gr_text "A4_POLARITY_SILK_v15-42" (at 130 78 0) (layer "Cmts.User")
+ (gr_text "A4_POLARITY_SILK_v15-42b" (at 130 78 0) (layer "Cmts.User")
   (effects (font (size 0.5 0.5) (thickness 0.08))))
- (gr_circle (center 136.1700 97.9300) (end 136.4500 97.9300) (stroke (width 0.12) (type default)) (fill solid) (layer "F.SilkS"))
- (gr_circle (center 143.5000 123.3900) (end 143.7200 123.3900) (stroke (width 0.12) (type default)) (fill solid) (layer "F.SilkS"))
- (gr_circle (center 125.6600 83.1800) (end 125.9100 83.1800) (stroke (width 0.12) (type default)) (fill solid) (layer "F.SilkS"))
- (gr_circle (center 125.6600 90.0800) (end 125.9100 90.0800) (stroke (width 0.12) (type default)) (fill solid) (layer "F.SilkS"))
- (gr_circle (center 114.0650 117.2000) (end 114.3150 117.2000) (stroke (width 0.12) (type default)) (fill solid) (layer "F.SilkS"))
- (gr_circle (center 136.8500 145.2250) (end 137.1300 145.2250) (stroke (width 0.12) (type default)) (fill solid) (layer "F.SilkS"))
- (gr_text "1" (at 136.8500 146.2250 0) (layer "F.SilkS")
-  (effects (font (size 0.55 0.55) (thickness 0.12))))
- (gr_circle (center 109.2300 84.2850) (end 109.4800 84.2850) (stroke (width 0.12) (type default)) (fill solid) (layer "F.SilkS"))
- (gr_circle (center 135.1900 84.2850) (end 135.4400 84.2850) (stroke (width 0.12) (type default)) (fill solid) (layer "F.SilkS"))
- (gr_line (start 119.6650 92.4250) (end 119.6650 93.4250) (stroke (width 0.12) (type default)) (layer "F.SilkS"))
- (gr_line (start 146.8050 91.8500) (end 146.8050 92.8500) (stroke (width 0.12) (type default)) (layer "F.SilkS"))
- (gr_line (start 113.5300 138.2200) (end 113.5300 139.3200) (stroke (width 0.12) (type default)) (layer "F.SilkS"))
- (gr_line (start 113.5300 142.2450) (end 113.5300 143.3450) (stroke (width 0.12) (type default)) (layer "F.SilkS"))
- (gr_line (start 124.1500 142.2450) (end 124.1500 143.3450) (stroke (width 0.12) (type default)) (layer "F.SilkS"))
- (gr_line (start 134.1800 142.2450) (end 134.1800 143.3450) (stroke (width 0.12) (type default)) (layer "F.SilkS"))
- (gr_line (start 124.6400 134.1200) (end 124.6400 135.2200) (stroke (width 0.12) (type default)) (layer "F.SilkS"))
- (gr_line (start 151.7800 107.9000) (end 151.7800 108.9000) (stroke (width 0.12) (type default)) (layer "F.SilkS"))
- (gr_text "A" (at 147.7300 108.4000 0) (layer "F.SilkS")
-  (effects (font (size 0.55 0.55) (thickness 0.12))))
- (gr_text "+" (at 131.1200 122.3450 0) (layer "F.SilkS")
-  (effects (font (size 0.7 0.7) (thickness 0.12))))
+ (gr_circle (center 135.6700 97.4300) (end 135.9500 97.4300) (stroke (width 0.15) (type default)) (fill solid) (layer "F.SilkS"))
+ (gr_circle (center 143.9500 122.9400) (end 144.1700 122.9400) (stroke (width 0.15) (type default)) (fill solid) (layer "F.SilkS"))
+ (gr_circle (center 125.0600 82.7300) (end 125.3100 82.7300) (stroke (width 0.15) (type default)) (fill solid) (layer "F.SilkS"))
+ (gr_circle (center 125.0600 89.6300) (end 125.3100 89.6300) (stroke (width 0.15) (type default)) (fill solid) (layer "F.SilkS"))
+ (gr_circle (center 113.4650 117.7000) (end 113.7150 117.7000) (stroke (width 0.15) (type default)) (fill solid) (layer "F.SilkS"))
+ (gr_circle (center 136.2500 144.0250) (end 136.5300 144.0250) (stroke (width 0.15) (type default)) (fill solid) (layer "F.SilkS"))
+ (gr_text "1" (at 136.2500 142.9250 0) (layer "F.SilkS")
+  (effects (font (size 0.8 0.8) (thickness 0.12))))
+ (gr_circle (center 108.6300 83.6850) (end 108.8800 83.6850) (stroke (width 0.15) (type default)) (fill solid) (layer "F.SilkS"))
+ (gr_circle (center 134.5900 83.6850) (end 134.8400 83.6850) (stroke (width 0.15) (type default)) (fill solid) (layer "F.SilkS"))
+ (gr_line (start 118.8650 92.4250) (end 118.8650 93.4250) (stroke (width 0.15) (type default)) (layer "F.SilkS"))
+ (gr_line (start 146.0050 91.8500) (end 146.0050 92.8500) (stroke (width 0.15) (type default)) (layer "F.SilkS"))
+ (gr_line (start 112.7800 138.2700) (end 112.7800 139.2700) (stroke (width 0.15) (type default)) (layer "F.SilkS"))
+ (gr_line (start 112.7800 142.2950) (end 112.7800 143.2950) (stroke (width 0.15) (type default)) (layer "F.SilkS"))
+ (gr_line (start 123.4000 142.2950) (end 123.4000 143.2950) (stroke (width 0.15) (type default)) (layer "F.SilkS"))
+ (gr_line (start 133.4300 142.2950) (end 133.4300 143.2950) (stroke (width 0.15) (type default)) (layer "F.SilkS"))
+ (gr_line (start 123.8900 134.1700) (end 123.8900 135.1700) (stroke (width 0.15) (type default)) (layer "F.SilkS"))
+ (gr_line (start 152.5800 107.9000) (end 152.5800 108.9000) (stroke (width 0.15) (type default)) (layer "F.SilkS"))
+ (gr_text "A" (at 147.0800 108.4000 0) (layer "F.SilkS")
+  (effects (font (size 0.8 0.8) (thickness 0.12))))
+ (gr_text "+" (at 131.7200 122.3450 0) (layer "F.SilkS")
+  (effects (font (size 0.85 0.85) (thickness 0.12))))
  (footprint "MountingHole_3.2mm" (layer "F.Cu") (at 103.5 83.5)
   (property "Reference" "H1" (at 0 -3 0) (layer "F.Fab") (effects (font (size 1 1) (thickness 0.15))))
